File: initial.sch (KiCad schematic (older format))
At the start: 1 part

Commit message: test
Parts:
- added D? (x2): LED, symbol LED
- added R? (x3): R, symbol R
Changed lines of the file:
@@
 LIBS:switches
 LIBS:relays
-LIBS:motors
 LIBS:transistors
 LIBS:conn
@@
 LIBS:contrib
 LIBS:valves
+LIBS:initial-cache
 EELAYER 25 0
 EELAYER END
@@
 	1    0    0    -1
 $EndComp
+$Comp
+L LED D?
+U 1 1 5C4B6AD0
+P 2000 2150
+F 0 "D?" H 2000 2250 50  0000 C CNN
+F 1 "LED" H 2000 2050 50  0000 C CNN
+F 2 "" H 2000 2150 50  0000 C CNN
+F 3 "" H 2000 2150 50  0000 C CNN
+	1    2000 2150
+	1    0    0    -1
+$EndComp
+$Comp
+L LED D?
+U 1 1 5C4B6B3F
+P 1950 2750
+F 0 "D?" H 1950 2850 50  0000 C CNN
+F 1 "LED" H 1950 2650 50  0000 C CNN
+F 2 "" H 1950 2750 50  0000 C CNN
+F 3 "" H 1950 2750 50  0000 C CNN
+	1    1950 2750
+	1    0    0    -1
+$EndComp
+$Comp
+L R R?
+U 1 1 5C4B6BFE
+P 3000 2800
+F 0 "R?" V 3080 2800 50  0000 C CNN
+F 1 "R" V 3000 2800 50  0000 C CNN
+F 2 "" V 2930 2800 50  0000 C CNN
+F 3 "" H 3000 2800 50  0000 C CNN
+	1    3000 2800
+	1    0    0    -1
+$EndComp
+$Comp
+L R R?
+U 1 1 5C4B6C1B
+P 3000 2150
+F 0 "R?" V 3080 2150 50  0000 C CNN
+F 1 "R" V 3000 2150 50  0000 C CNN
+F 2 "" V 2930 2150 50  0000 C CNN
+F 3 "" H 3000 2150 50  0000 C CNN
+	1    3000 2150
+	1    0    0    -1
+$EndComp
+$Comp
+L R R?
+U 1 1 5C4B6F3B
+P 32700 8650
+F 0 "R?" V 32780 8650 50  0000 C CNN
+F 1 "R" V 32700 8650 50  0000 C CNN
+F 2 "" V 32630 8650 50  0000 C CNN
+F 3 "" H 32700 8650 50  0000 C CNN
+	1    32700 8650
+	1    0    0    -1
+$EndComp

Commit message: passes erc
Parts:
- removed R?: R, symbol R
- removed RV?: POT, symbol POT
- added J1: Conn 2x5, symbol Connector_Generic:Conn_02x05_Odd_Even
- R1, R2: renamed from R?; value R -> 200
- gave numbers to parts that had none: 2
Connections:
- net at D2.1 (K): now also R2.1
- net at D2.2 (A): now also J1.3 (Pin_3)
- net at D1.1 (K): now also R1.1
- net at D1.2 (A): now also J1.1 (Pin_1)
- net at R1.2: now also R2.2, J1.9 (Pin_9)
- no-connect marks 0 -> 7
Other:
- note added: "3v3\nGPOI2\nGPOI3\nGPOI4\nGND"
- note added: "5v\n5v\nGND\nGPOI14\nGPOI15"
Changed lines of the file:
@@
-EESchema Schematic File Version 2
+EESchema Schematic File Version 4
 LIBS:power
 LIBS:device
-LIBS:switches
-LIBS:relays
-LIBS:transistors
-LIBS:conn
-LIBS:linear
-LIBS:regul
 LIBS:74xx
-LIBS:cmos4000
-LIBS:adc-dac
-LIBS:memory
-LIBS:xilinx
-LIBS:microcontrollers
-LIBS:dsp
-LIBS:microchip
-LIBS:analog_switches
-LIBS:motorola
-LIBS:texas
-LIBS:intel
 LIBS:audio
 LIBS:interface
-LIBS:digital-audio
-LIBS:philips
-LIBS:display
-LIBS:cypress
-LIBS:siliconi
-LIBS:opto
-LIBS:atmel
-LIBS:contrib
-LIBS:valves
 LIBS:initial-cache
-EELAYER 25 0
+EELAYER 26 0
 EELAYER END
 $Descr A4 11693 8268
@@
 $EndDescr
 $Comp
-L POT RV?
-U 1 1 5C408E2A
-P -677750 -368500
-F 0 "RV?" V -677925 -368500 50  0000 C CNN
-F 1 "POT" V -677850 -368500 50  0000 C CNN
-F 2 "" H -677750 -368500 50  0001 C CNN
-F 3 "" H -677750 -368500 50  0001 C CNN
-	1    -677750 -368500
+L LED D2
+U 1 1 5C4B6AD0
+P 4300 3850
+F 0 "D2" H 4300 3950 50  0000 C CNN
+F 1 "LED" H 4300 3750 50  0000 C CNN
+F 2 "" H 4300 3850 50  0000 C CNN
+F 3 "" H 4300 3850 50  0000 C CNN
+	1    4300 3850
+	0    -1   -1   0
+$EndComp
+$Comp
+L LED D1
+U 1 1 5C4B6B3F
+P 3800 3850
+F 0 "D1" H 3800 3950 50  0000 C CNN
+F 1 "LED" H 3800 3750 50  0000 C CNN
+F 2 "" H 3800 3850 50  0000 C CNN
+F 3 "" H 3800 3850 50  0000 C CNN
+	1    3800 3850
+	0    -1   -1   0
+$EndComp
+$Comp
+L R R1
+U 1 1 5C4B6BFE
+P 3800 4600
+F 0 "R1" V 3880 4600 50  0000 C CNN
+F 1 "200" V 3800 4600 50  0000 C CNN
+F 2 "" V 3730 4600 50  0000 C CNN
+F 3 "" H 3800 4600 50  0000 C CNN
+	1    3800 4600
 	1    0    0    -1
 $EndComp
 $Comp
-L GND #PWR?
-U 1 1 5C408E5B
-P -677750 -368200
-F 0 "#PWR?" H -677750 -368450 50  0001 C CNN
-F 1 "GND" H -677750 -368350 50  0000 C CNN
-F 2 "" H -677750 -368200 50  0001 C CNN
-F 3 "" H -677750 -368200 50  0001 C CNN
-	1    -677750 -368200
+L R R2
+U 1 1 5C4B6C1B
+P 4300 4600
+F 0 "R2" V 4380 4600 50  0000 C CNN
+F 1 "200" V 4300 4600 50  0000 C CNN
+F 2 "" V 4230 4600 50  0000 C CNN
+F 3 "" H 4300 4600 50  0000 C CNN
+	1    4300 4600
 	1    0    0    -1
 $EndComp
 $Comp
-L LED D?
-U 1 1 5C4B6AD0
-P 2000 2150
-F 0 "D?" H 2000 2250 50  0000 C CNN
-F 1 "LED" H 2000 2050 50  0000 C CNN
-F 2 "" H 2000 2150 50  0000 C CNN
-F 3 "" H 2000 2150 50  0000 C CNN
-	1    2000 2150
+L Connector_Generic:Conn_02x05_Odd_Even J1
+U 1 1 5C4E6805
+P 5700 4300
+F 0 "J1" H 5750 4717 50  0000 C CNN
+F 1 "Conn 2x5" H 5750 4626 50  0000 C CNN
+F 2 "" H 5700 4300 50  0001 C CNN
+F 3 "~" H 5700 4300 50  0001 C CNN
+	1    5700 4300
 	1    0    0    -1
 $EndComp
-$Comp
-L LED D?
-U 1 1 5C4B6B3F
-P 1950 2750
-F 0 "D?" H 1950 2850 50  0000 C CNN
-F 1 "LED" H 1950 2650 50  0000 C CNN
-F 2 "" H 1950 2750 50  0000 C CNN
-F 3 "" H 1950 2750 50  0000 C CNN
-	1    1950 2750
-	1    0    0    -1
-$EndComp
-$Comp
-L R R?
-U 1 1 5C4B6BFE
-P 3000 2800
-F 0 "R?" V 3080 2800 50  0000 C CNN
-F 1 "R" V 3000 2800 50  0000 C CNN
-F 2 "" V 2930 2800 50  0000 C CNN
-F 3 "" H 3000 2800 50  0000 C CNN
-	1    3000 2800
-	1    0    0    -1
-$EndComp
-$Comp
-L R R?
-U 1 1 5C4B6C1B
-P 3000 2150
-F 0 "R?" V 3080 2150 50  0000 C CNN
-F 1 "R" V 3000 2150 50  0000 C CNN
-F 2 "" V 2930 2150 50  0000 C CNN
-F 3 "" H 3000 2150 50  0000 C CNN
-	1    3000 2150
-	1    0    0    -1
-$EndComp
-$Comp
-L R R?
-U 1 1 5C4B6F3B
-P 32700 8650
-F 0 "R?" V 32780 8650 50  0000 C CNN
-F 1 "R" V 32700 8650 50  0000 C CNN
-F 2 "" V 32630 8650 50  0000 C CNN
-F 3 "" H 32700 8650 50  0000 C CNN
-	1    32700 8650
-	1    0    0    -1
-$EndComp
+Wire Wire Line
+	3800 4050 3800 4450
+Wire Wire Line
+	4300 4050 4300 4450
+Wire Wire Line
+	3800 4750 3800 4900
+Wire Wire Line
+	3800 4900 4300 4900
+Wire Wire Line
+	4300 4900 4300 4750
+Text Notes 4950 4450 0    50   ~ 0
+3v3\nGPOI2\nGPOI3\nGPOI4\nGND
+Wire Wire Line
+	4300 4900 5500 4900
+Wire Wire Line
+	5500 4900 5500 4500
+Connection ~ 4300 4900
+NoConn ~ 5500 4400
+NoConn ~ 5500 4300
+Wire Wire Line
+	3800 3500 5350 3500
+Wire Wire Line
+	5350 3500 5350 4100
+Wire Wire Line
+	5350 4100 5500 4100
+Wire Wire Line
+	4300 3650 5300 3650
+Wire Wire Line
+	5300 3650 5300 4200
+Wire Wire Line
+	5300 4200 5500 4200
+Wire Wire Line
+	3800 3500 3800 3650
+NoConn ~ 6000 4100
+NoConn ~ 6000 4200
+NoConn ~ 6000 4300
+NoConn ~ 6000 4400
+NoConn ~ 6000 4500
+Text Notes 6250 4500 0    50   ~ 0
+5v\n5v\nGND\nGPOI14\nGPOI15
 $EndSCHEMATC
